File: PCB/LedDisplay.brd (EAGLE design)
At the start: 104 x 54 mm, 32 parts, among them IC1 AT90S2313S, IC2 74164D, IC3 74164D, IC4 74164D

Commit message: Updated pcb dimensions. Now is fits perfectly to the casing. Also some of the elements were changed to DIP packages.
Parts:
- removed IC1: AT90S2313S, atmel:SO20L
- added C1, C2: (no value), capacitor-wima:C2.5-3
- added IC6: AT90S2313P, atmel:DIL20
- added IC7: 74HC595D, 74xx-eu:SO16
- added Q1: (no value), crystal:HC49U70
- added S1: (no value), switch-omron:B3F-10XX
- moved R24 281.3 mm to (13.3, 43.6), turned to 180 degrees
- moved R23 269.9 mm to (16.0, 35.6), turned to 180 degrees
- moved R22 267.5 mm to (22.2, 35.6)
- moved R20 265.6 mm to (27.6, 43.5), turned to 180 degrees
- moved R16 254.7 mm to (44.3, 43.6), turned to 180 degrees
- moved R14 251.6 mm to (54.2, 43.5)
- moved R21 250.0 mm to (25.0, 19.0), turned to 180 degrees
- moved R15 245.7 mm to (46.9, 35.5), turned to 180 degrees
- moved R17 244.2 mm to (20.0, 43.5), turned to 180 degrees
- moved R12 241.5 mm to (59.8, 35.5), turned to 180 degrees
- moved R13 230.5 mm to (59.1, 11.2), turned to 180 degrees
- moved R19 230.2 mm to (19.8, 11.6), turned to 180 degrees
- moved R18 227.2 mm to (14.7, 19.0)
- moved R9 223.8 mm to (53.5, 35.5), turned to 180 degrees
- moved R11 217.3 mm to (52.7, 11.1), turned to 180 degrees
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Connections:
- new net N$1: IC7.7, U$4.8
- new net N$2: IC7.6, U$4.7
- new net N$3: IC7.5, U$4.6
- new net N$4: IC7.4, U$4.5
- new net N$5: IC7.3, U$4.4
- new net N$57: C1.2, IC6.4, Q1.2
- new net N$58: C2.2, IC6.5, Q1.1
- new net N$59: IC6.2
- new net N$6: IC7.2, U$4.3
- new net N$60: IC6.3
- new net N$61: IC2.9, IC3.9, IC4.9, IC6.8
- new net N$62: IC2.1, IC2.2, IC6.9
- new net N$63: IC2.8, IC3.8, IC4.8, IC6.11
- new net N$64: IC6.6, S1.1
- new net N$65: IC6.7
- new net N$7: IC7.1, U$4.2
- new net N$74: IC6.12, IC7.12
- new net N$75: IC6.13, IC7.10
- new net N$76: IC6.14, IC7.11
- new net N$77: IC6.15, IC7.14
- new net N$8: IC7.15, U$4.1
- net GND: now also C1.1, C2.1, IC6.10, IC7.8, U$4.9; no longer IC1.10
- net N$24: now also IC4.1, IC4.2
- net N$40: now also IC3.1, IC3.2
- net VCC: now also IC6.20, IC7.16; no longer IC1.20
Routing:
- net N$68: track 0.00 -> 155.1 mm
- net N$72: track 0.00 -> 124.4 mm
- net N$67: track 0.00 -> 123.3 mm
- net N$66: track 0.00 -> 111.4 mm
- net N$73: track 0.00 -> 101.6 mm
- net N$69: track 0.00 -> 91.4 mm
- net N$70: track 0.00 -> 90.7 mm
- net N$74: track 0.00 -> 27.1 mm
- net N$7: track 0.00 -> 22.2 mm
- net N$75: track 0.00 -> 21.1 mm
- net N$6: track 0.00 -> 20.4 mm
- net N$76: track 0.00 -> 18.7 mm
- net N$56: track 0.00 -> 18.7 mm
- net N$5: track 0.00 -> 18.3 mm
- net N$4: track 0.00 -> 16.6 mm
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Other:
- board size 104 x 54 mm -> 104 x 50 mm

Commit message: Another part of improvements in pcb layout, especially on the top layer.
Parts:
- added R25: 0, resistor:M1206
- moved R4 10.4 mm to (93.0, 34.8), turned to 180 degrees
- moved R8 9.79 mm to (76.5, 43.4)
- moved R5 9.69 mm to (92.7, 20.6), turned to 270 degrees
- moved R13 9.17 mm to (60.9, 20.2), turned to 270 degrees
- moved R2 8.94 mm to (81.6, 18.8), turned to 180 degrees
- moved R7 8.43 mm to (76.0, 34.9), turned to 0 degrees
- moved R17 7.96 mm to (21.2, 35.6)
- moved R20 7.88 mm to (27.5, 35.6)
- moved R22 7.75 mm to (22.2, 43.4)
- moved IC2 5.73 mm to (84.8, 26.4), turned to 0 degrees
- moved R6 3.92 mm to (85.2, 43.3), turned to 0 degrees
- moved R10 2.29 mm to (44.4, 11.2)
- moved R21 1.65 mm to (26.7, 19.0)
- moved R1 1.63 mm to (84.5, 34.8)
- moved R23 1.14 mm to (14.9, 35.6)
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Connections:
- new net N$78: R25.2, U$1.8, U$4.12
- net N$68: now also R25.1; no longer U$1.8, U$4.12
Routing:
- net N$71: track 0.00 -> 141.4 mm
- net N$61: track 0.00 -> 111.7 mm
- net N$63: track 0.00 -> 98.6 mm
- net N$24: track 0.00 -> 64.4 mm
- net N$40: track 0.00 -> 50.3 mm
- net GND: track 8.80 -> 56.7 mm
- net N$21: track 0.00 -> 44.6 mm
- net N$37: track 0.00 -> 44.5 mm
- net N$53: track 0.00 -> 43.6 mm
- net N$78: track 0.00 -> 35.0 mm
- net N$68: track 155.1 -> 121.4 mm
- net N$33: track 0.00 -> 22.6 mm
- net N$17: track 0.00 -> 20.6 mm
- net N$38: track 0.00 -> 19.1 mm
- net N$34: track 0.00 -> 19.0 mm
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